File: pcb/eagle/powermeter-shunt/powermeter.sch (EAGLE design)
At the start: 29 parts, among them IC1 INA126P, IC2 LM324N, IC3 MCP3208, IC4 MEA1D0512SC

Commit message: Made design compatible with MCP3204 (can now use MCP3204 or MCP3208)
Parts:
- added SV2: (no value), con-lstb:MA03-1
Connections:
- removed net N$10: IC3.CH0, R7.1
- removed net VSAMPLE: IC3.CH1, R8.1
- new net VM1: IC3.CH1, R8.1, SV2.2
- new net VM2: IC3.CH0, R7.1, SV2.3
- net GND: now also IC3.CH6, SV2.1
Other:
- note added: "Connecting Channel 6 to GND allows for using MCP3204 instead of MCP 3208. Channel 6 of MCP 3208 is DGND of MCP 3204. Other pins as compatible."
Changed lines of the file:
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@@
 <part name="P+2" library="supply1" deviceset="+12V" device=""/>
 <part name="GND18" library="supply1" deviceset="GND" device=""/>
+<part name="SV2" library="con-lstb" deviceset="MA03-1" device=""/>
+<part name="GND19" library="supply1" deviceset="GND" device=""/>
+<part name="GND20" library="supply1" deviceset="GND" device=""/>
 </parts>
 <sheets>
@@
 (min. 10 % of the rated load) to meet
 the specifications.</text>
+<text x="149.86" y="-119.38" size="1.778" layer="91">Connecting Channel 6 to GND allows
+for using MCP3204 instead of MCP 3208.
+Channel 6 of MCP 3208 is DGND of MCP 3204.
+Other pins as compatible.</text>
 </plain>
 <instances>
@@
 <instance part="P+2" gate="1" x="137.16" y="63.5"/>
 <instance part="GND18" gate="1" x="137.16" y="25.4"/>
+<instance part="SV2" gate="G$1" x="210.82" y="55.88"/>
+<instance part="GND19" gate="1" x="223.52" y="45.72"/>
+<instance part="GND20" gate="1" x="167.64" y="-104.14"/>
 </instances>
 <busses>
@@
 <wire x1="137.16" y1="35.56" x2="137.16" y2="27.94" width="0.1524" layer="91"/>
 <pinref part="GND18" gate="1" pin="GND"/>
+</segment>
+<segment>
+<pinref part="SV2" gate="G$1" pin="1"/>
+<wire x1="218.44" y1="53.34" x2="223.52" y2="53.34" width="0.1524" layer="91"/>
+<wire x1="223.52" y1="53.34" x2="223.52" y2="48.26" width="0.1524" layer="91"/>
+<pinref part="GND19" gate="1" pin="GND"/>
+</segment>
+<segment>
+<pinref part="GND20" gate="1" pin="GND"/>
+<wire x1="167.64" y1="-101.6" x2="167.64" y2="-93.98" width="0.1524" layer="91"/>
+<pinref part="IC3" gate="G$1" pin="CH6"/>
+<wire x1="167.64" y1="-93.98" x2="177.8" y2="-93.98" width="0.1524" layer="91"/>
 </segment>
 </net>
@@
 </segment>
 </net>
-<net name="N$10" class="0">
+<net name="VM2" class="0">
 <segment>
 <pinref part="R7" gate="G$1" pin="1"/>
 <pinref part="IC3" gate="G$1" pin="CH0"/>
-<wire x1="172.72" y1="-63.5" x2="177.8" y2="-63.5" width="0.1524" layer="91"/>
-</segment>
-</net>
-<net name="VSAMPLE" class="0">
+<wire x1="172.72" y1="-63.5" x2="175.26" y2="-63.5" width="0.1524" layer="91"/>
+<wire x1="175.26" y1="-63.5" x2="177.8" y2="-63.5" width="0.1524" layer="91"/>
+<wire x1="175.26" y1="-63.5" x2="175.26" y2="-48.26" width="0.1524" layer="91"/>
+<wire x1="175.26" y1="-48.26" x2="182.88" y2="-48.26" width="0.1524" layer="91"/>
+<label x="182.88" y="-48.26" size="1.778" layer="95" xref="yes"/>
+<junction x="175.26" y="-63.5"/>
+</segment>
+<segment>
+<pinref part="SV2" gate="G$1" pin="3"/>
+<wire x1="218.44" y1="58.42" x2="223.52" y2="58.42" width="0.1524" layer="91"/>
+<label x="223.52" y="58.42" size="1.778" layer="95" xref="yes"/>
+</segment>
+</net>
+<net name="VM1" class="0">
 <segment>
 <pinref part="IC3" gate="G$1" pin="CH1"/>
@@
 <label x="195.58" y="-17.78" size="1.778" layer="95" xref="yes"/>
 </segment>
-</net>
+<segment>
+<pinref part="SV2" gate="G$1" pin="2"/>
+<wire x1="218.44" y1="55.88" x2="236.22" y2="55.88" width="0.1524" layer="91"/>
+<label x="236.22" y="55.88" size="1.778" layer="95" xref="yes"/>
+</segment>
+</net>
